File: youdbetterrun.kicad_pcb (KiCad board)
At the start: 4 copper layers, 60 x 53 mm, 48 parts, among them J201 GT-USB-7010ASV, J301 Conn_01x05_Pin, J302 Conn_01x10_Pin, J401 FH12A-24S-0.5SH(55), Q201 S8050, Q202 S8050, Q401 Q_NMOS_GSD, SW301 TS-1088R-02026, SW302 TS-1088R-02026, U202 CP2104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

Commit message: Rename project
Damn squatters
Parts:
- J201: footprint busbuddy:USB_C_Receptacle_G-Switch_GT-USB-7010ASV -> youdbetterrun:USB_C_Receptacle_G-Switch_GT-USB-7010ASV
- L401: footprint busbuddy:L_4x4x2.6 -> youdbetterrun:L_4x4x2.6
- SW301, SW302: footprint busbuddy:TS-1088R-02026_SW_SMD_3x4mm -> youdbetterrun:TS-1088R-02026_SW_SMD_3x4mm
Changed lines of the file:
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@@
 		)
 	)
-	(footprint "busbuddy:L_4x4x2.6"
+	(footprint "youdbetterrun:L_4x4x2.6"
 		(layer "F.Cu")
 		(at 97 101.25 90)
@@
 			)
 		)
-		(property "Footprint" "busbuddy:L_4x4x2.6"
+		(property "Footprint" "youdbetterrun:L_4x4x2.6"
 			(at 0 0 90)
 			(unlocked yes)
@@
 		)
 	)
-	(footprint "busbuddy:USB_C_Receptacle_G-Switch_GT-USB-7010ASV"
+	(footprint "youdbetterrun:USB_C_Receptacle_G-Switch_GT-USB-7010ASV"
 		(layer "F.Cu")
 		(at 149 68 90)
@@
 			)
 		)
-		(property "Footprint" "busbuddy:USB_C_Receptacle_G-Switch_GT-USB-7010ASV"
+		(property "Footprint" "youdbetterrun:USB_C_Receptacle_G-Switch_GT-USB-7010ASV"
 			(at 0 0 90)
 			(unlocked yes)
@@
 		)
 	)
-	(footprint "busbuddy:TS-1088R-02026_SW_SMD_3x4mm"
+	(footprint "youdbetterrun:TS-1088R-02026_SW_SMD_3x4mm"
 		(layer "F.Cu")
 		(at 134 82.5 90)
@@
 			)
 		)
-		(property "Footprint" "busbuddy:TS-1088R-02026_SW_SMD_3x4mm"
+		(property "Footprint" "youdbetterrun:TS-1088R-02026_SW_SMD_3x4mm"
 			(at 0 0 90)
 			(unlocked yes)
@@
 		)
 	)
-	(footprint "busbuddy:TS-1088R-02026_SW_SMD_3x4mm"
+	(footprint "youdbetterrun:TS-1088R-02026_SW_SMD_3x4mm"
 		(layer "F.Cu")
 		(at 138 82.5 90)
@@
 			)
 		)
-		(property "Footprint" "busbuddy:TS-1088R-02026_SW_SMD_3x4mm"
+		(property "Footprint" "youdbetterrun:TS-1088R-02026_SW_SMD_3x4mm"
 			(at 0 0 90)
 			(unlocked yes)

Commit message: Add OSHW logo
Parts:
- added REF**: OSHW_LOGO, youdbetterrun:OSHW_LOGO, F.Cu at (132.6, 94.1)
Other:
- board text added: "You'd Better Run Rev B © 2024 Marcel Robitaille"
- board text removed: "EPD Driver Rev A © 2024 Marcel Robitaille"
