File: epd.kicad_sch (KiCad schematic)
At the start: 19 parts, among them J4 FH12A-24S-0.5SH(55), Q3 Q_NMOS_GSD

Commit message: Switch to ESP32
Parts:
- Q3: symbol Device:Q_NMOS_GSD -> Transistor_FET:Q_NMOS_GSD
Other:
- company: (none) -> Marcel Robitaille
- title: (none) -> EPD
Changed lines of the file:
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@@
 	(generator_version "9.0")
 	(paper "A4")
+	(title_block
+		(title "EPD")
+		(company "Marcel Robitaille")
+	)
 	(junction
 		(at 45.72 76.2)
@@
 	)
 	(symbol
-		(lib_id "Device:Q_NMOS_GSD")
+		(lib_id "Transistor_FET:Q_NMOS_GSD")
 		(at 83.82 86.36 0)
 		(unit 1)
@@
 		(fields_autoplaced yes)
 		(property "Reference" "Q3"
-			(at 90.17 85.09 0)
+			(at 90.17 85.0899 0)
 			(effects
 				(font
@@
 		)
 		(property "Value" "Q_NMOS_GSD"
-			(at 90.17 87.63 0)
-			(effects
-				(font
+			(at 90.17 87.6299 0)
+			(effects
+				(font
