File: ldo.kicad_sch (KiCad schematic)
At the start: 4 parts, among them U3 SPX3819M5-L-3-3

Commit message: Switch to ESP32
Other:
- company: (none) -> Marcel Robitaille
- title: (none) -> LDO
Changed lines of the file:
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@@
 	(generator_version "9.0")
 	(paper "A5")
+	(title_block
+		(title "LDO")
+		(company "Marcel Robitaille")
+	)
 	(junction
 		(at 72.39 60.96)
